File: li-ion_charging.kicad_sch (KiCad schematic)
At the start: 13 parts, among them J1 Conn_01x02, J7 Jack-DC, U11 DW01A, U3 MCP73812T-420I-OT

Commit message: General Layout Complete
Completed general layout, beginning to add debugging components such as test points and
Parts:
- U14: value ~ -> (none)
