File: V1/PCB/Peripheral.kicad_sch (KiCad schematic)
At the start: 52 parts, among them J10 Conn_01x03, J11 Conn_01x03, J12 Conn_01x03, J13 Conn_01x03, J2 Conn_01x04, J3 Conn_01x06, J4 Conn_01x06, J5 Conn_01x06, J6 Conn_01x07, J9 Conn_01x03

Commit message: Updated/Verified Values
Other:
- note added: "Reset Pin needs to be pulled up"
Changed lines of the file:
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@@
+		)
+	)
+	(text "Reset Pin needs to be pulled up"
+		(exclude_from_sim no)
+		(at 180.848 56.896 0)
+		(effects
+			(font
+				(size 0.635 0.635)
+			)
 		)
 	)
