File: V1/PCB/Power.kicad_sch (KiCad schematic)
At the start: 67 parts, among them U10 TPS63002, U2 TPS63001, U8 TPS63002

Commit message: Updated/Verified Values
Parts:
- L1, L2, L3, L4: value 6.8uH -> 2.2uH
Changed lines of the file:
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@@
 			)
 		)
-		(property "Value" "6.8uH"
+		(property "Value" "2.2uH"
 			(at 44.45 183.134 90)
 			(show_name no)
@@
 			)
 		)
-		(property "Value" "6.8uH"
+		(property "Value" "2.2uH"
 			(at 44.45 119.634 90)
 			(show_name no)
@@
 			)
 		)
-		(property "Value" "6.8uH"
+		(property "Value" "2.2uH"
 			(at 44.45 151.384 90)
 			(show_name no)
@@
 			)
 		)
-		(property "Value" "6.8uH"
+		(property "Value" "2.2uH"
 			(at 44.45 86.614 90)
 			(show_name no)
